File: V1/eumesmo-rl-4ch12a-v1.kicad_pcb (KiCad board)
At the start: 2 copper layers, 53 x 67.8 mm, 25 parts, among them J1 250-202, J2 250-204, J3 DB142V-5.08-4P, J4 DB142V-5.08-4P, K1 G5PZ-1A, K2 G5PZ-1A, K3 G5PZ-1A, K4 G5PZ-1A

Commit message: Adjusted version number
Other:
- board text added: "V1.2 2026-06-13"
- board text added: "eumesmo-rl-4ch12a-v1"
- board text removed: "RELAY-24V-4CH-12A-V1"
- board text removed: "V1.1 2026-06-02"
Changed lines of the file:
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@@
 	(paper "A4")
 	(title_block
-		(title "4x 24V Relay Module")
-		(date "2026-06-02")
-		(rev "V1.1")
+		(title "eumesmo 4x 24V 12A Relay Module")
+		(date "2026-06-13")
+		(rev "V1.2")
 	)
 	(layers
@@
 		(property ki_fp_filters "Connector*:*_1x??_*")
 		(sheetname "/")
-		(sheetfile "relay-24v-4ch-12a-v1.kicad_sch")
+		(sheetfile "eumesmo-rl-4ch12a-v1.kicad_sch")
 		(units
 			(unit
@@
 		(property ki_fp_filters "LED* LED_SMD:* LED_THT:*")
 		(sheetname "/")
-		(sheetfile "relay-24v-4ch-12a-v1.kicad_sch")
+		(sheetfile "eumesmo-rl-4ch12a-v1.kicad_sch")
 		(units
 			(unit
@@
 		(property ki_fp_filters "TO-???* *_Diode_* *SingleDiode* D_*")
 		(sheetname "/")
-		(sheetfile "relay-24v-4ch-12a-v1.kicad_sch")
+		(sheetfile "eumesmo-rl-4ch12a-v1.kicad_sch")
 		(units
 			(unit
@@
 		(property ki_fp_filters "LED* LED_SMD:* LED_THT:*")
 		(sheetname "/")
-		(sheetfile "relay-24v-4ch-12a-v1.kicad_sch")
+		(sheetfile "eumesmo-rl-4ch12a-v1.kicad_sch")
 		(units
 			(unit
@@
 		(property ki_fp_filters "Relay*SPST*Omron*G5PZ*")
 		(sheetname "/")
-		(sheetfile "relay-24v-4ch-12a-v1.kicad_sch")
+		(sheetfile "eumesmo-rl-4ch12a-v1.kicad_sch")
 		(units
 			(unit
@@
 		(property ki_fp_filters "R_*")
 		(sheetname "/")
-		(sheetfile "relay-24v-4ch-12a-v1.kicad_sch")
+		(sheetfile "eumesmo-rl-4ch12a-v1.kicad_sch")
 		(units
 			(unit
@@
 		(property ki_fp_filters "TO-???* *_Diode_* *SingleDiode* D_*")
 		(sheetname "/")
-		(sheetfile "relay-24v-4ch-12a-v1.kicad_sch")
+		(sheetfile "eumesmo-rl-4ch12a-v1.kicad_sch")
 		(units
 			(unit
@@
 		(property ki_fp_filters "RV_* Varistor*")
 		(sheetname "/")
-		(sheetfile "relay-24v-4ch-12a-v1.kicad_sch")
+		(sheetfile "eumesmo-rl-4ch12a-v1.kicad_sch")
 		(units
 			(unit
@@
 		(property ki_fp_filters "Connector*:*_1x??_*")
 		(sheetname "/")
-		(sheetfile "relay-24v-4ch-12a-v1.kicad_sch")
+		(sheetfile "eumesmo-rl-4ch12a-v1.kicad_sch")
 		(units
 			(unit
@@
 		(property ki_fp_filters "R_*")
 		(sheetname "/")
-		(sheetfile "relay-24v-4ch-12a-v1.kicad_sch")
+		(sheetfile "eumesmo-rl-4ch12a-v1.kicad_sch")
 		(units
 			(unit
@@
 		(property ki_fp_filters "TO-???* *_Diode_* *SingleDiode* D_*")
 		(sheetname "/")
-		(sheetfile "relay-24v-4ch-12a-v1.kicad_sch")
+		(sheetfile "eumesmo-rl-4ch12a-v1.kicad_sch")
 		(units
 			(unit
@@
 		(property ki_fp_filters "Relay*SPST*Omron*G5PZ*")
 		(sheetname "/")
-		(sheetfile "relay-24v-4ch-12a-v1.kicad_sch")
+		(sheetfile "eumesmo-rl-4ch12a-v1.kicad_sch")
 		(units
 			(unit
@@
 		(property ki_fp_filters "RV_* Varistor*")
 		(sheetname "/")
-		(sheetfile "relay-24v-4ch-12a-v1.kicad_sch")
+		(sheetfile "eumesmo-rl-4ch12a-v1.kicad_sch")
 		(units
 			(unit
@@
 		(property ki_fp_filters "RV_* Varistor*")
 		(sheetname "/")
-		(sheetfile "relay-24v-4ch-12a-v1.kicad_sch")
+		(sheetfile "eumesmo-rl-4ch12a-v1.kicad_sch")
 		(units
 			(unit
@@
 		(property ki_fp_filters "Connector*:*_1x??_*")
 		(sheetname "/")
-		(sheetfile "relay-24v-4ch-12a-v1.kicad_sch")
+		(sheetfile "eumesmo-rl-4ch12a-v1.kicad_sch")
 		(units
 			(unit
@@
 		(property ki_fp_filters "Relay*SPST*Omron*G5PZ*")
 		(sheetname "/")
-		(sheetfile "relay-24v-4ch-12a-v1.kicad_sch")
+		(sheetfile "eumesmo-rl-4ch12a-v1.kicad_sch")
 		(units
 			(unit
@@
 		(property ki_fp_filters "R_*")
 		(sheetname "/")
-		(sheetfile "relay-24v-4ch-12a-v1.kicad_sch")
+		(sheetfile "eumesmo-rl-4ch12a-v1.kicad_sch")
 		(units
 			(unit
@@
 		(property ki_fp_filters "LED* LED_SMD:* LED_THT:*")
 		(sheetname "/")
-		(sheetfile "relay-24v-4ch-12a-v1.kicad_sch")
+		(sheetfile "eumesmo-rl-4ch12a-v1.kicad_sch")
 		(units
 			(unit
@@
 		(property ki_fp_filters "TO-???* *_Diode_* *SingleDiode* D_*")
 		(sheetname "/")
-		(sheetfile "relay-24v-4ch-12a-v1.kicad_sch")
+		(sheetfile "eumesmo-rl-4ch12a-v1.kicad_sch")
 		(units
 			(unit
@@
 		(property ki_fp_filters "Relay*SPST*Omron*G5PZ*")
 		(sheetname "/")
-		(sheetfile "relay-24v-4ch-12a-v1.kicad_sch")
+		(sheetfile "eumesmo-rl-4ch12a-v1.kicad_sch")
 		(units
 			(unit
@@
 		(property ki_fp_filters "RV_* Varistor*")
 		(sheetname "/")
-		(sheetfile "relay-24v-4ch-12a-v1.kicad_sch")
+		(sheetfile "eumesmo-rl-4ch12a-v1.kicad_sch")
 		(units
 			(unit
@@
 		(property ki_fp_filters "Connector*:*_1x??_*")
 		(sheetname "/")
-		(sheetfile "relay-24v-4ch-12a-v1.kicad_sch")
+		(sheetfile "eumesmo-rl-4ch12a-v1.kicad_sch")
 		(units
 			(unit
@@
 		(property ki_fp_filters "R_*")
 		(sheetname "/")
-		(sheetfile "relay-24v-4ch-12a-v1.kicad_sch")
+		(sheetfile "eumesmo-rl-4ch12a-v1.kicad_sch")
 		(units
 			(unit
@@
 		(property ki_fp_filters "LED* LED_SMD:* LED_THT:*")
 		(sheetname "/")
-		(sheetfile "relay-24v-4ch-12a-v1.kicad_sch")
+		(sheetfile "eumesmo-rl-4ch12a-v1.kicad_sch")
 		(units
 			(unit
@@
 		(layer "Edge.Cuts")
 	)
-	(gr_text "V1.1\n2026-06-02"
+	(gr_text "V1.2\n2026-06-13"
 		(at 128.5 70.5 90)
 		(layer "F.SilkS")
@@
 		)
 	)
-	(gr_text "RELAY-24V-4CH-12A-V1"
+	(gr_text "eumesmo-rl-4ch12a-v1"
 		(at 137 64.25 0)
 		(layer "F.SilkS")

Commit message: Adjusted product name on the silkscreen
Other:
- board text added: "eumesmo-rl-4ch12a"
- board text removed: "eumesmo-rl-4ch12a-v1"
Changed lines of the file:
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@@
 		)
 	)
-	(gr_text "eumesmo-rl-4ch12a-v1"
+	(gr_text "eumesmo-rl-4ch12a"
 		(at 137 64.25 0)
 		(layer "F.SilkS")

Commit message: Release V1.2.0
Other:
- board text added: "V1.2 2026-06-17"
- board text removed: "V1.2 2026-06-13"
Changed lines of the file:
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@@
 		)
-	)
-	(gr_rect
-		(start 126 67.75)
-		(end 128.75 73.25)
-		(stroke
-			(width 0.1)
-			(type solid)
-		)
-		(fill no)
-		(layer "F.SilkS")
 	)
 	(gr_line
@@
 	)
 	(gr_rect
+		(start 175.75 101.75)
+		(end 177.25 109.25)
+		(stroke
+			(width 0.1)
+			(type solid)
+		)
+		(fill no)
+		(layer "F.SilkS")
+	)
+	(gr_rect
 		(start 125 62.2)
 		(end 178 130)
@@
 		(layer "Edge.Cuts")
 	)
-	(gr_text "V1.2\n2026-06-13"
-		(at 128.5 70.5 90)
+	(gr_text "V1.2 2026-06-17"
+		(at 176.5 105.5 90)
 		(layer "F.SilkS")
 		(effects
@@
 				(thickness 0.1)
 			)
-			(justify bottom)
-		)
-	)
+		)
+	)
